File: pcb_main/rebote-smd.kicad_pcb (KiCad board)
At the start: 2 copper layers, 55.5 x 100 mm, 66 parts, among them J1 V+ GND, J2 NMJ6HCD2, J3 NMJ6HCD2, J4 V+ GND, SW1 SW_3PDT, U1 TL072, U2 L78L05_SOT89, U3 PT2399

Commit message: Updates to template
Other:
- board text added: "TKW 2023 rev ${GIT_VERSION}"
- board text removed: "TKW 2023 rev 0.1"
Changed lines of the file:
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@@
     )
   )
+  (property "GIT_VERSION" "v0.0.1")
   (net 0 "")
   (net 1 "GND")
@@
     )
   )
-  (gr_text "TKW 2023 rev 0.1" (at 122.01 96.05 90) (layer "F.SilkS")
+  (gr_text "TKW 2023 rev ${GIT_VERSION}" (at 122.01 96.05 90) (layer "F.SilkS")
     (effects (font (size 1 1) (thickness 0.15) italic) (justify left bottom))
   )
